Commit message: Add a four wheel differential drive robot

File: src/my_robot/urdf/my_robot.xacro (robot description, xacro)
@@ -31,4 +31,5 @@
       </geometry>
     </visual>
+<!--
     <collision name='back_caster_collision'>
       <origin xyz="-0.15 0 -0.05" rpy=" 0 0 0"/>
@@ -54,65 +55,133 @@
         <sphere radius="0.05"/>
       </geometry>
-    </visual>
-  </link>
-  <!-- Left wheel -->
-  <link name='left_wheel'>
-    <collision name='left_wheel_collision'>
-      <origin xyz="0 0 0" rpy="0 1.5707 1.5707"/>
-      <geometry>
-	<cylinder radius="0.1" length="0.05"/>
-      </geometry>
-    </collision>
-    <visual name='left_wheel_visual'>
-      <origin xyz="0 0 0" rpy="0 1.5707 1.5707"/>
-      <geometry>
-	<cylinder radius="0.1" length="0.05"/>
-      </geometry>
-    </visual>
-    <inertial>
-      <mass value="5"/>
-      <origin xyz="0 0 0" rpy="0 1.5707 1.5707"/>
-      <inertia
-          ixx="0.1" ixy="0" ixz="0"
-          iyy="0.1" iyz="0"
-          izz="0.1"
-      />
-    </inertial>
-  </link>
-  <joint type="continuous" name="left_wheel_hinge">
-    <origin xyz="0 0.15 0" rpy="0 0 0"/>
-    <child link="left_wheel"/>
-    <parent link="chassis"/>
-    <axis xyz="0 1 0" rpy="0 0 0"/>
-    <limit effort="10000" velocity="1000"/>
-    <dynamics damping="1.0" friction="1.0"/>
-  </joint>
-  <!-- Right wheel -->
-  <link name='right_wheel'>
-    <collision name='right_wheel_collision'>
-      <origin xyz="0 0 0" rpy="0 1.5707 1.5707"/>
-      <geometry>
-	<cylinder radius="0.1" length="0.05"/>
-      </geometry>
-    </collision>
-    <visual name='right_wheel_visual'>
-      <origin xyz="0 0 0" rpy="0 1.5707 1.5707"/>
-      <geometry>
-	<cylinder radius="0.1" length="0.05"/>
-      </geometry>
-    </visual>
-    <inertial>
-      <mass value="5"/>
-      <origin xyz="0 0 0" rpy="0 1.5707 1.5707"/>
-      <inertia
-          ixx="0.1" ixy="0" ixz="0"
-          iyy="0.1" iyz="0"
-          izz="0.1"
-      />
-    </inertial>
-  </link>
-  <joint type="continuous" name="right_wheel_hinge">
-    <origin xyz="0 -0.15 0" rpy="0 0 0"/>
-    <child link="right_wheel"/>
+    </visual> -->
+  </link>
+  <!-- Front Left wheel -->
+  <link name='front_left_wheel'>
+    <collision name='front_left_wheel_collision'>
+      <origin xyz="0 0 0" rpy="0 1.5707 1.5707"/>
+      <geometry>
+	<cylinder radius="0.1" length="0.05"/>
+      </geometry>
+    </collision>
+    <visual name='front_left_wheel_visual'>
+      <origin xyz="0 0 0" rpy="0 1.5707 1.5707"/>
+      <geometry>
+	<cylinder radius="0.1" length="0.05"/>
+      <material name = "Green"/>
+      </geometry>
+    </visual>
+    <inertial>
+      <mass value="5"/>
+      <origin xyz="0 0 0" rpy="0 1.5707 1.5707"/>
+      <inertia
+          ixx="0.1" ixy="0" ixz="0"
+          iyy="0.1" iyz="0"
+          izz="0.1"
+      />
+    </inertial>
+  </link>
+  <joint type="continuous" name="front_left_wheel_hinge">
+    <origin xyz="0.15 0.15 0" rpy="0 0 0"/>
+    <child link="front_left_wheel"/>
+    <parent link="chassis"/>
+    <axis xyz="0 1 0" rpy="0 0 0"/>
+    <limit effort="10000" velocity="1000"/>
+    <dynamics damping="1.0" friction="1.0"/>
+  </joint>
+    <!-- Front Right wheel -->
+  <link name='front_right_wheel'>
+    <collision name='front_right_wheel_collision'>
+      <origin xyz="0 0 0" rpy="0 1.5707 1.5707"/>
+      <geometry>
+	<cylinder radius="0.1" length="0.05"/>
+      </geometry>
+    </collision>
+    <visual name='front_right_wheel_visual'>
+      <origin xyz="0 0 0" rpy="0 1.5707 1.5707"/>
+      <geometry>
+	<cylinder radius="0.1" length="0.05"/>
+  <material name = "Green"/>
+      </geometry>
+    </visual>
+    <inertial>
+      <mass value="5"/>
+      <origin xyz="0 0 0" rpy="0 1.5707 1.5707"/>
+      <inertia
+          ixx="0.1" ixy="0" ixz="0"
+          iyy="0.1" iyz="0"
+          izz="0.1"
+      />
+    </inertial>
+  </link>
+  <joint type="continuous" name="front_right_wheel_hinge">
+    <origin xyz="0.15 -0.15 0" rpy="0 0 0"/>
+    <child link="front_right_wheel"/>
+    <parent link="chassis"/>
+    <axis xyz="0 1 0" rpy="0 0 0"/>
+    <limit effort="10000" velocity="1000"/>
+    <dynamics damping="1.0" friction="1.0"/>
+  </joint>
+<!-- Rear Left wheel -->
+  <link name='rear_left_wheel'>
+    <collision name='rear_left_wheel_collision'>
+      <origin xyz="0 0 0" rpy="0 1.5707 1.5707"/>
+      <geometry>
+	<cylinder radius="0.1" length="0.05"/>
+  <material name = "Green"/>
+      </geometry>
+    </collision>
+    <visual name='rear_left_wheel_visual'>
+      <origin xyz="0 0 0" rpy="0 1.5707 1.5707"/>
+      <geometry>
+	<cylinder radius="0.1" length="0.05"/>
+      </geometry>
+    </visual>
+    <inertial>
+      <mass value="5"/>
+      <origin xyz="0 0 0" rpy="0 1.5707 1.5707"/>
+      <inertia
+          ixx="0.1" ixy="0" ixz="0"
+          iyy="0.1" iyz="0"
+          izz="0.1"
+      />
+    </inertial>
+  </link>
+  <joint type="continuous" name="rear_left_wheel_hinge">
+    <origin xyz="-0.15 0.15 0" rpy="0 0 0"/>
+    <child link="rear_left_wheel"/>
+    <parent link="chassis"/>
+    <axis xyz="0 1 0" rpy="0 0 0"/>
+    <limit effort="10000" velocity="1000"/>
+    <dynamics damping="1.0" friction="1.0"/>
+  </joint>
+  <!-- Rear Right wheel -->
+  <link name='rear_right_wheel'>
+    <collision name='rear_right_wheel_collision'>
+      <origin xyz="0 0 0" rpy="0 1.5707 1.5707"/>
+      <geometry>
+	<cylinder radius="0.1" length="0.05"/>
+      </geometry>
+    </collision>
+    <visual name='rear_right_wheel_visual'>
+      <origin xyz="0 0 0" rpy="0 1.5707 1.5707"/>
+      <geometry>
+	<cylinder radius="0.1" length="0.05"/>
+  <material name = "Green"/>
+      </geometry>
+    </visual>
+    <inertial>
+      <mass value="5"/>
+      <origin xyz="0 0 0" rpy="0 1.5707 1.5707"/>
+      <inertia
+          ixx="0.1" ixy="0" ixz="0"
+          iyy="0.1" iyz="0"
+          izz="0.1"
+      />
+    </inertial>
+  </link>
+  <joint type="continuous" name="rear_right_wheel_hinge">
+    <origin xyz="-0.15 -0.15 0" rpy="0 0 0"/>
+    <child link="rear_right_wheel"/>
     <parent link="chassis"/>
     <axis xyz="0 1 0" rpy="0 0 0"/>
@@ -181,10 +250,10 @@
   </joint>
   <!-- Material -->
-  <gazebo reference="left_wheel">
+  <!-- <gazebo reference="left_wheel">
     <material>Gazebo/Green</material>
   </gazebo>
   <gazebo reference="right_wheel">
     <material>Gazebo/Green</material>
-  </gazebo>
+  </gazebo> -->
   <gazebo reference="chassis">
     <material>Gazebo/Blue</material>

Commit message: Create skid steeering drive robot

File: src/my_robot/urdf/my_robot.xacro (robot description, xacro)
@@ -31,29 +31,4 @@
       </geometry>
     </visual>
-<!--
-    <collision name='back_caster_collision'>
-      <origin xyz="-0.15 0 -0.05" rpy=" 0 0 0"/>
-      <geometry>
-        <sphere radius="0.0499"/>
-      </geometry>
-    </collision>
-    <visual name='back_caster_visual'>
-      <origin xyz="-0.15 0 -0.05" rpy=" 0 0 0"/>
-      <geometry>
-        <sphere radius="0.05"/>
-      </geometry>
-    </visual>
-    <collision name='front_caster_collision'>
-      <origin xyz="0.15 0 -0.05" rpy=" 0 0 0"/>
-      <geometry>
-        <sphere radius="0.0499"/>
-      </geometry>
-    </collision>
-    <visual name='front_caster_visual'>
-      <origin xyz="0.15 0 -0.05" rpy=" 0 0 0"/>
-      <geometry>
-        <sphere radius="0.05"/>
-      </geometry>
-    </visual> -->
   </link>
   <!-- Front Left wheel -->
@@ -69,5 +44,4 @@
       <geometry>
 	<cylinder radius="0.1" length="0.05"/>
-      <material name = "Green"/>
       </geometry>
     </visual>
@@ -88,5 +62,5 @@
     <axis xyz="0 1 0" rpy="0 0 0"/>
     <limit effort="10000" velocity="1000"/>
-    <dynamics damping="1.0" friction="1.0"/>
+    <dynamics damping="1.0" friction="0.5"/>
   </joint>
     <!-- Front Right wheel -->
@@ -102,5 +76,4 @@
       <geometry>
 	<cylinder radius="0.1" length="0.05"/>
-  <material name = "Green"/>
       </geometry>
     </visual>
@@ -121,5 +94,5 @@
     <axis xyz="0 1 0" rpy="0 0 0"/>
     <limit effort="10000" velocity="1000"/>
-    <dynamics damping="1.0" friction="1.0"/>
+    <dynamics damping="1.0" friction="0.5"/>
   </joint>
 <!-- Rear Left wheel -->
@@ -129,5 +102,4 @@
       <geometry>
 	<cylinder radius="0.1" length="0.05"/>
-  <material name = "Green"/>
       </geometry>
     </collision>
@@ -154,5 +126,5 @@
     <axis xyz="0 1 0" rpy="0 0 0"/>
     <limit effort="10000" velocity="1000"/>
-    <dynamics damping="1.0" friction="1.0"/>
+    <dynamics damping="1.0" friction="0.5"/>
   </joint>
   <!-- Rear Right wheel -->
@@ -168,5 +140,4 @@
       <geometry>
 	<cylinder radius="0.1" length="0.05"/>
-  <material name = "Green"/>
       </geometry>
     </visual>
@@ -187,5 +158,5 @@
     <axis xyz="0 1 0" rpy="0 0 0"/>
     <limit effort="10000" velocity="1000"/>
-    <dynamics damping="1.0" friction="1.0"/>
+    <dynamics damping="1.0" friction="0.5"/>
   </joint>
   <!-- camera -->
@@ -250,15 +221,21 @@
   </joint>
   <!-- Material -->
-  <!-- <gazebo reference="left_wheel">
-    <material>Gazebo/Green</material>
-  </gazebo>
-  <gazebo reference="right_wheel">
-    <material>Gazebo/Green</material>
-  </gazebo> -->
+  <gazebo reference="front_left_wheel_visual">
+    <material>Gazebo/Grey</material>
+  </gazebo>
+  <gazebo reference="front_right_wheel_visual">
+    <material>Gazebo/Grey</material>
+  </gazebo>
+    <gazebo reference="rear_left_wheel_visual">
+    <material>Gazebo/Grey</material>
+  </gazebo>
+  <gazebo reference="rear_right_wheel_visual">
+    <material>Gazebo/Grey</material>
+  </gazebo>
   <gazebo reference="chassis">
-    <material>Gazebo/Blue</material>
+    <material>Gazebo/Red</material>
   </gazebo>
   <gazebo reference="camera">
-    <material>Gazebo/Red</material>
+    <material>Gazebo/DarkYellow</material>
   </gazebo>
 </robot>

Commit message: Change the color of the robot

File: src/my_robot/urdf/my_robot.xacro (robot description, xacro)
@@ -182,14 +182,14 @@
   <!-- Material -->
   <gazebo reference="left_wheel">
-    <material>Gazebo/Green</material>
+    <material>Gazebo/Grey</material>
   </gazebo>
   <gazebo reference="right_wheel">
-    <material>Gazebo/Green</material>
+    <material>Gazebo/Grey</material>
   </gazebo>
   <gazebo reference="chassis">
-    <material>Gazebo/Blue</material>
+    <material>Gazebo/Red</material>
   </gazebo>
   <gazebo reference="camera">
-    <material>Gazebo/Red</material>
+    <material>Gazebo/DarkYellow</material>
   </gazebo>
 </robot>

Commit message: Change the wheel dimensions of the robot

File: src/my_robot/urdf/my_robot.xacro (robot description, xacro)
@@ -61,5 +61,5 @@
       <origin xyz="0 0 0" rpy="0 1.5707 1.5707"/>
       <geometry>
-	<cylinder radius="0.1" length="0.05"/>
+	<cylinder radius="0.11" length="0.055"/>
       </geometry>
     </collision>
@@ -67,5 +67,5 @@
       <origin xyz="0 0 0" rpy="0 1.5707 1.5707"/>
       <geometry>
-	<cylinder radius="0.1" length="0.05"/>
+	<cylinder radius="0.11" length="0.055"/>
       </geometry>
     </visual>
@@ -93,5 +93,5 @@
       <origin xyz="0 0 0" rpy="0 1.5707 1.5707"/>
       <geometry>
-	<cylinder radius="0.1" length="0.05"/>
+	<cylinder radius="0.11" length="0.055"/>
       </geometry>
     </collision>
@@ -99,5 +99,5 @@
       <origin xyz="0 0 0" rpy="0 1.5707 1.5707"/>
       <geometry>
-	<cylinder radius="0.1" length="0.05"/>
+	<cylinder radius="0.11" length="0.055"/>
       </geometry>
     </visual>

Commit message: Corrent the wheel dimensions

File: src/my_robot/urdf/my_robot.xacro (robot description, xacro)
@@ -61,5 +61,5 @@
       <origin xyz="0 0 0" rpy="0 1.5707 1.5707"/>
       <geometry>
-	<cylinder radius="0.11" length="0.055"/>
+	<cylinder radius="0.1" length="0.05"/>
       </geometry>
     </collision>
@@ -67,5 +67,5 @@
       <origin xyz="0 0 0" rpy="0 1.5707 1.5707"/>
       <geometry>
-	<cylinder radius="0.11" length="0.055"/>
+	<cylinder radius="0.1" length="0.05"/>
       </geometry>
     </visual>
@@ -93,5 +93,5 @@
       <origin xyz="0 0 0" rpy="0 1.5707 1.5707"/>
       <geometry>
-	<cylinder radius="0.11" length="0.055"/>
+	<cylinder radius="0.1" length="0.05"/>
       </geometry>
     </collision>
@@ -99,5 +99,5 @@
       <origin xyz="0 0 0" rpy="0 1.5707 1.5707"/>
       <geometry>
-	<cylinder radius="0.11" length="0.055"/>
+	<cylinder radius="0.1" length="0.05"/>
       </geometry>
     </visual>

Commit message: Add RGBD camera to my_robot

File: src/my_robot/urdf/my_robot.xacro (robot description, xacro)
@@ -144,5 +144,5 @@
     </inertial>
   </link>
-  <joint type="fixed" name="camera_joint">
+  <joint name="camera_joint" type="fixed">
     <origin xyz="0.2 0 0" rpy="0 0 0"/>
     <child link="camera"/>
@@ -150,5 +150,13 @@
     <axis xyz="0 1 0"/>
   </joint>
-  <!-- hokuyo -->
+    <!-- RGBD camera -->
+  <link name="camera_link_optical">
+  </link>
+  <joint name="camera_optical_joint" type="fixed">
+    <origin xyz="0 0 0" rpy="-1.5707 0 -1.5707"/>
+    <parent link="camera"/>
+    <child link="camera_link_optical"/>
+  </joint>
+  <!-- hokuyo Lidar -->
   <link name='hokuyo'>
     <collision name="hokuyo_collision">
